File: kicad_files/f169_fullplate.kicad_pcb (KiCad board)
At the start: 2 copper layers, 347.6 x 137 mm, 1 part

Commit message: Update connector area with a more solid outline. New renders pending
Other:
- outline, holes or cut-outs redrawn
