File: kicad_files/f169_halfplate.kicad_pcb (KiCad board)
At the start: 2 copper layers, 347.6 x 137 mm, 0 parts

Commit message: Added inscription and renamed files
Parts:
- added G***: LOGO, f169_plates_graphics:half_plate_inscription, F.Cu at (332.0, 145.5)

Commit message: Update connector area with a more solid outline. New renders pending
Other:
- outline, holes or cut-outs redrawn
